File: hardware/readout_64x64/readout_64x64_regulated.kicad_pcb (KiCad board)
At the start: 4 copper layers, 91.9 x 56.3 mm, 66 parts, among them IC1 74LVC595APW, IC10 ADG732BSUZ, IC11 LM358BAIDR, IC12 AD7476ARTZ, IC13 AD7476ARTZ, IC14 LM358BAIDR, IC2 74LVC595APW, IC3 74LVC595APW, IC4 74LVC595APW, IC5 74LVC595APW, IC6 74LVC595APW, IC7 74LVC595APW, IC8 74LVC595APW, IC9 ADG732BSUZ, J1 5051107091, J2 5051107091, SW2 SW_MEC_5E, U1 Teensy4.1, U6 LM2776

Commit message: Readout board: MCP41HV51 potentiometers assembled by the board house; JLCPCB assembly files
- VR1, VR2 (MCP41HV51-103E/ST): no longer do-not-populate; LCSC C637062 added (schematic and layout)
- Layout synced to the schematic: TP9 do-not-populate, IC11/IC14 value TLV9362
- Gerbers, JLCPCB BOM and placement files re-exported with the Fabrication Toolkit plugin (KiCad 10)
- Copper and nets unchanged; ERC/DRC results unchanged from before the edit
Parts:
- IC11, IC14: value LM358BAIDR -> TLV9362
Changed lines of the file:
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@@
 		(sheetname "/")
 		(sheetfile "readout_64x64_regulated.kicad_sch")
-		(attr exclude_from_pos_files)
+		(attr exclude_from_pos_files dnp)
 		(fp_line
 			(start -0.7 -0.7)
@@
 			)
 		)
-		(property "Value" "LM358BAIDR"
+		(property "Value" "TLV9362"
 			(at 0 0 90)
 			(layer "F.SilkS")
@@
 			)
 		)
-		(property "Value" "LM358BAIDR"
+		(property "Value" "TLV9362"
 			(at 0 0 90)
 			(layer "F.SilkS")
@@
 			)
 		)
+		(property "LCSC Part #" "C637062"
+			(at 0 0 90)
+			(unlocked yes)
+			(layer "F.Fab")
+			(hide yes)
+			(effects
+				(font
+					(size 1 1)
+					(thickness 0.15)
+				)
+			)
+		)
 		(sheetname "/")
 		(sheetfile "readout_64x64_regulated.kicad_sch")
-		(attr smd dnp)
+		(attr smd)
 		(fp_line
 			(start -3.675 -2.525)
@@
 			)
 		)
+		(property "LCSC Part #" "C637062"
+			(at 0 0 90)
+			(unlocked yes)
+			(layer "F.Fab")
+			(hide yes)
+			(effects
+				(font
+					(size 1 1)
+					(thickness 0.15)
+				)
+			)
+		)
 		(sheetname "/")
 		(sheetfile "readout_64x64_regulated.kicad_sch")
-		(attr smd dnp)
+		(attr smd)
 		(fp_line
 			(start -3.675 -2.525)
