File: hardware/readout_64x64/readout_64x64_regulated.kicad_sch (KiCad schematic)
At the start: 68 parts, among them IC1 74LVC595APW, IC10 ADG732BSUZ, IC11 TLV9362, IC12 AD7476ARTZ, IC13 AD7476ARTZ, IC14 TLV9362, IC2 74LVC595APW, IC3 74LVC595APW, IC4 74LVC595APW, IC5 74LVC595APW, IC6 74LVC595APW, IC7 74LVC595APW, IC8 74LVC595APW, IC9 ADG732BSUZ, J1 5051107091, J2 5051107091, SW2 SW_MEC_5E, U1 Teensy4.1, U6 LM2776

Commit message: Readout board: MCP41HV51 potentiometers assembled by the board house; JLCPCB assembly files
- VR1, VR2 (MCP41HV51-103E/ST): no longer do-not-populate; LCSC C637062 added (schematic and layout)
- Layout synced to the schematic: TP9 do-not-populate, IC11/IC14 value TLV9362
- Gerbers, JLCPCB BOM and placement files re-exported with the Fabrication Toolkit plugin (KiCad 10)
- Copper and nets unchanged; ERC/DRC results unchanged from before the edit
Parts:
- VR1, VR2: LCSC Part # (none) -> C637062; now fitted
Changed lines of the file:
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@@
 		(in_bom yes)
 		(on_board yes)
-		(dnp yes)
+		(dnp no)
 		(property "Reference" "VR2"
 			(at 300.482 225.298 0)
@@
 			)
 		)
+		(property "LCSC Part #" "C637062"
+			(at 314.96 205.74 0)
+			(effects
+				(font
+					(size 1.27 1.27)
+				)
+				(hide yes)
+			)
+		)
 		(pin "13"
 		)
@@
 		(in_bom yes)
 		(on_board yes)
-		(dnp yes)
+		(dnp no)
 		(property "Reference" "VR1"
 			(at 224.282 225.298 0)
@@
 				(hide yes)
 			)
+		)
+		(property "LCSC Part #" "C637062"
+			(at 238.76 205.74 0)
+			(effects
+				(font
+					(size 1.27 1.27)
+				)
+				(hide yes)
+			)

Commit message: Readout board: SW2 tactile switch from JLCPCB's assembly library (TS4538TP, C398052)
Fits the existing PTS647 footprint (same 4.5 x 4.5 mm body and terminals); only the part number fields change.
Assembly files re-exported; ERC/DRC unchanged.
Parts:
- SW2: LCSC Part # C2689502 -> C398052; Manufacturer_Part_Number (none) -> TS4538TP
Changed lines of the file:
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@@
 			)
 		)
-		(property "LCSC Part #" "C2689502"
+		(property "LCSC Part #" "C398052"
 			(at 358.14 152.4 0)
 			(effects
+				(font
+					(size 1.27 1.27)
+				)
+				(hide yes)
+			)
+		)
+		(property "Manufacturer_Part_Number" "TS4538TP"
+			(at 358.14 152.4 0)
+			(effects
